File: KiCad_Lock/KiCad_Lock.kicad_sch (KiCad schematic)
At the start: 3 parts, among them M1 Stepper_Motor_unipolar_5pin, U1 ProS3

Commit message: hej
Other:
- note added: "5V"
- note added: "A"
- note added: "B"
- note added: "C"
- note added: "D"
- note added: "Driver Board"
- note added: "ESP32 ProS3"
- note added: "Stepper Motor"
- moved on the sheet: U1, U2
