File: KiCad_Lock/KiCad_Lock.kicad_sch (KiCad schematic)
At the start: 3 parts, among them M1 Stepper_Motor_unipolar_5pin, U1 ProS3

Commit message: yo
Parts:
- U1: footprint AndreasLibrary:ESP32-PROS3 -> PCM_Espressif:ESP32-PROS3
- U2: footprint (none) -> Connector_PinSocket_2.54mm:PinSocket_1x06_P2.54mm_Vertical
Changed lines of the file:
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@@
 			)
 		)
-		(property "Footprint" ""
+		(property "Footprint" "Connector_PinSocket_2.54mm:PinSocket_1x06_P2.54mm_Vertical"
 			(at 167.64 93.98 0)
 			(effects
@@
 			)
 		)
-		(property "Footprint" "AndreasLibrary:ESP32-PROS3"
+		(property "Footprint" "PCM_Espressif:ESP32-PROS3"
 			(at 144.272 97.282 0)
 			(effects
