File: KiCad_Nem_Laas/KiCad_Nem_Laas.kicad_pcb (KiCad board)
At the start: 2 copper layers, 6 parts, among them SW1 SW_Push, U1 ProS3

Commit message: asdaw
Routing:
- net Net-(U1-IO14): track 23.6 -> 24.4 mm
Changed lines of the file:
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@@
 		(tags "resistor handsolder")
 		(property "Reference" "R1"
-			(at 0 -1.5 360)
+			(at 0 -1.5 0)
 			(layer "F.SilkS")
 			(effects
@@
 		)
 		(property "Value" "220"
-			(at 0 1.5 360)
+			(at 0 1.5 0)
 			(layer "F.Fab")
 			(effects
@@
 		)
 		(fp_text user "${REFERENCE}"
-			(at 0 0 360)
+			(at 0 0 0)
 			(layer "F.Fab")
 			(effects
@@
 		(tags "LED handsolder")
 		(property "Reference" "D1"
-			(at 0 -1.43 360)
+			(at 0 -1.43 0)
 			(layer "F.SilkS")
 			(effects
@@
 		)
 		(property "Value" "LED"
-			(at 0 1.43 360)
+			(at 0 1.43 0)
 			(layer "F.Fab")
 			(effects
@@
 		)
 		(fp_text user "${REFERENCE}"
-			(at 0 0 360)
+			(at 0 0 0)
 			(layer "F.Fab")
 			(effects
@@
 		(tags "resistor handsolder")
 		(property "Reference" "R2"
-			(at 0 -1.17 360)
+			(at 0 -1.17 0)
 			(layer "F.SilkS")
 			(effects
@@
 		)
 		(property "Value" "220"
-			(at 0 1.17 360)
+			(at 0 1.17 0)
 			(layer "F.Fab")
 			(effects
@@
 		)
 		(fp_text user "${REFERENCE}"
-			(at 0 0 360)
+			(at 0 0 0)
 			(layer "F.Fab")
 			(effects
@@
 		(tags "LED handsolder")
 		(property "Reference" "D2"
-			(at 0 -1.5 360)
+			(at 0 -1.5 0)
 			(layer "F.SilkS")
 			(effects
@@
 		)
 		(property "Value" "LED"
-			(at 0 1.43 360)
+			(at 0 1.43 0)
 			(layer "F.Fab")
 			(effects
@@
 		)
 		(fp_text user "${REFERENCE}"
-			(at 0 0 360)
+			(at 0 0 0)
 			(layer "F.Fab")
 			(effects
@@
 	(segment
 		(start 152.395 97.415)
-		(end 168.31 81.5)
+		(end 152.395 96.105)
 		(width 0.5)
 		(layer "F.Cu")
@@
 	)
 	(segment
-		(start 168.31 81.5)
+		(start 152.395 96.105)
+		(end 167 81.5)
+		(width 0.5)
+		(layer "F.Cu")
+		(net 3)
+	)
+	(segment
+		(start 167 81.5)
 		(end 169.4025 81.5)
 		(width 0.5)
@@
 	)
 	(segment
-		(start 166.85 85.5)
+		(start 168.5 85.5)
 		(end 169.4025 85.5)
 		(width 0.5)
@@
 	)
 	(segment
-		(start 154.935 97.415)
-		(end 166.85 85.5)
+		(start 157.5 94.5)
+		(end 159.5 94.5)
 		(width 0.5)
 		(layer "F.Cu")
+		(net 4)
+	)
+	(segment
+		(start 154.935 97.415)
+		(end 154.935 97.065)
+		(width 0.5)
+		(layer "F.Cu")
+		(net 4)
+	)
+	(segment
+		(start 154.935 97.065)
+		(end 157.5 94.5)
+		(width 0.5)
+		(layer "F.Cu")
+		(net 4)
+	)
+	(segment
+		(start 159.5 94.5)
+		(end 168.5 85.5)
+		(width 0.5)
+		(layer "F.Cu")
