File: KiCad_Fjernbetjening/KiCad_Nem_Laas.kicad_pcb (KiCad board)
At the start: 2 copper layers, 6 parts, among them SW1 SW_Push, U1 ProS3

Commit message: yo
Routing:
- net Net-(U1-IO4): track 41.6 -> 42.4 mm
Changed lines of the file:
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@@
 	)
 	(segment
-		(start 135.5 96.53)
-		(end 134.615 97.415)
-		(width 0.5)
-		(layer "F.Cu")
-		(net 5)
-	)
-	(segment
-		(start 135.5 93)
-		(end 135.5 96.53)
+		(start 134.5 92.75)
+		(end 134.5 97.3)
 		(width 0.5)
 		(layer "F.Cu")
@@
 		(net 5)
 	)
+	(segment
+		(start 134.5 97.3)
+		(end 134.615 97.415)
+		(width 0.5)
+		(layer "F.Cu")
+		(net 5)
+	)
 	(via
-		(at 135.5 93)
+		(at 134.5 92.75)
 		(size 0.6)
 		(drill 0.3)
@@
 	)
 	(segment
-		(start 168 90)
-		(end 138.5 90)
+		(start 137.25 90)
+		(end 168 90)
 		(width 0.5)
 		(layer "B.Cu")
@@
 	)
 	(segment
-		(start 138.5 90)
-		(end 135.5 93)
+		(start 134.5 92.75)
+		(end 137.25 90)
 		(width 0.5)
 		(layer "B.Cu")
